File: IoTGW_Isolation/IoTGW_Isolation.kicad_sch (KiCad schematic)
At the start: 33 parts, among them J1 39502-1008, J4 39502-1008, Q1 Q_PMOS, U1 TEA1-0505, U2 ISO1452BDWR, U3 LTV-817S, U4 LTV-817S, U5 LTV-817S, U6 LTV-817S, U7 LTV-817S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

Commit message: PCB routing update
Connections:
- net GPIO_COMM: now also J4.7 (Pin_7); no longer J4.6 (Pin_6)
- net GPIO_R: now also J4.6 (Pin_6); no longer J4.7 (Pin_7)
- net RS-485_A renamed RS-485_+
- net RS-485_B renamed RS-485_-
Other:
- note added: "A"
- note added: "B"
Changed lines of the file:
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@@
 	(wire
 		(pts
-			(xy 39.37 115.57) (xy 49.53 115.57)
+			(xy 39.37 115.57) (xy 50.8 115.57)
 		)
 		(stroke
@@
 	(wire
 		(pts
-			(xy 39.37 102.87) (xy 49.53 102.87)
+			(xy 39.37 102.87) (xy 50.8 102.87)
 		)
 		(stroke
@@
 		)
 	)
+	(text "B"
+		(exclude_from_sim no)
+		(at 130.81 46.99 0)
+		(effects
+			(font
+				(size 1.27 1.27)
+			)
+		)
+	)
 	(text "I think we dont need it at all: Cost inneffective."
 		(exclude_from_sim no)
@@
 		)
 	)
+	(text "A"
+		(exclude_from_sim no)
+		(at 130.81 44.45 0)
+		(effects
+			(font
+				(size 1.27 1.27)
+			)
+		)
+	)
 	(text "SUPPORTS HALF AND FULL DUPLEX"
 		(exclude_from_sim no)
@@
 		)
 	)
-	(label "RS-485_B"
+	(label "RS-485_-"
 		(at 59.69 105.41 0)
 		(fields_autoplaced yes)
@@
 		)
 	)
-	(label "RS-485_A"
+	(label "RS-485_+"
 		(at 59.69 102.87 0)
 		(fields_autoplaced yes)
@@
 		)
 	)
-	(label "RS-485_A"
-		(at 49.53 102.87 180)
+	(label "RS-485_+"
+		(at 50.8 102.87 180)
 		(fields_autoplaced yes)
 		(effects
@@
 		)
 	)
-	(label "RS-485_B"
-		(at 49.53 115.57 180)
+	(label "RS-485_-"
+		(at 50.8 115.57 180)
 		(fields_autoplaced yes)
 		(effects
@@
 		)
 	)
+	(global_label "GPIO_COMM"
+		(shape input)
+		(at 101.6 46.99 180)
+		(fields_autoplaced yes)
+		(effects
+			(font
+				(size 0.889 0.889)
+				(color 0 0 0 1)
+			)
+			(justify right)
+		)
+		(property "Intersheetrefs" "${INTERSHEET_REFS}"
+			(at 91.8483 46.99 0)
+			(effects
+				(font
+					(size 1.27 1.27)
+				)
+				(justify right)
+				(hide yes)
+			)
+		)
+	)
 	(global_label "GPIO_EXT_2"
 		(shape output)
@@
 		)
 	)
+	(global_label "GPIO_R"
+		(shape output)
+		(at 101.6 44.45 180)
+		(fields_autoplaced yes)
+		(effects
+			(font
+				(size 0.889 0.889)
+				(color 0 0 0 1)
+			)
+			(justify right)
+		)
+		(property "Intersheetrefs" "${INTERSHEET_REFS}"
+			(at 94.8116 44.45 0)
+			(effects
+				(font
+					(size 1.27 1.27)
+				)
+				(justify right)
+				(hide yes)
+			)
+		)
+	)
 	(global_label "GPIO_EXT_2"
 		(shape input)
@@
 		)
 	)
-	(global_label "RS-485_B"
+	(global_label "RS-485_-"
 		(shape output)
 		(at 120.65 46.99 0)
@@
 		)
 		(property "Intersheetrefs" "${INTERSHEET_REFS}"
-			(at 129.6823 46.99 0)
+			(at 129.894 46.99 0)
 			(effects
 				(font
@@
 		)
 	)
-	(global_label "RS-485_A"
+	(global_label "RS-485_+"
 		(shape output)
 		(at 120.65 44.45 0)
@@
 		)
 		(property "Intersheetrefs" "${INTERSHEET_REFS}"
-			(at 129.5553 44.45 0)
+			(at 129.894 44.45 0)
 			(effects
 				(font
@@
 				(hide yes)
 			)
-		)
-	)
-	(global_label "GPIO_COMM"
-		(shape input)
-		(at 101.6 44.45 180)
-		(fields_autoplaced yes)
-		(effects
-			(font
-				(size 0.889 0.889)
-				(color 0 0 0 1)
-			)
-			(justify right)
-		)
-		(property "Intersheetrefs" "${INTERSHEET_REFS}"
-			(at 91.8483 44.45 0)
-			(effects
-				(font
-					(size 1.27 1.27)
-				)
-				(justify right)
-				(hide yes)
-			)
-		)
-	)
-	(global_label "GPIO_R"
-		(shape output)
-		(at 101.6 46.99 180)
-		(fields_autoplaced yes)
-		(effects
-			(font
-				(size 0.889 0.889)
-				(color 0 0 0 1)
-			)
-			(justify right)
-		)
-		(property "Intersheetrefs" "${INTERSHEET_REFS}"
-			(at 94.8116 46.99 0)
-			(effects
-				(font
-					(size 1.27 1.27)
-				)
-				(justify right)
-				(hide yes)
-			)
