File: IoTGW_Isolation/IoTGW_Isolation.kicad_sch (KiCad schematic)
At the start: 38 parts, among them J1 39502-1009, J2 39502-1009, Q1 Q_PMOS, U1 TEA1-0505, U2 NCP1117-3.3, U3 LTV-817S, U4 LTV-817S, U5 LTV-817S, U6 LTV-817S, U7 LTV-817S, U8 LTV-817S, U9 ISO1452BDWR

Commit message: FInal PCB, plot, dimensions, 3D step file
Parts:
- removed F1, F2: Polyfuse, Fuse:Fuse_0805_2012Metric, symbol Device:Polyfuse
- removed Q1: Q_PMOS, symbol Device:Q_PMOS_GSD
- removed R1: 10k, symbol Device:R
- removed U1: TEA1-0505, Converter_DCDC:Converter_DCDC_TRACO_TEA1-xxxx_THT, symbol Converter_DCDC:TEA1-0505
- added C6: 22uF, Capacitor_SMD:C_0805_2012Metric_Pad1.18x1.45mm_HandSolder, symbol Device:C_Polarized
- added U10: TBA2-0511, Converter_DCDC:Converter_DCDC_TRACO_TBA2-xxxx_Single_THT, symbol Converter_DCDC:TBA2-0511
- R10, R2, R3, R4, R8, R9: value 110R -> 120R
Connections:
- net 3.3V_CONN is gone; now on net +3.3V_OUT: J2.9 (Pin_9)
- net 5V_CONN is gone; now on net +5V_OUT: J2.8 (Pin_8)
- net +5V: now also C6.1, U10.1 (+Vin)
- net +5V_OUT: now also U10.6 (+Vout)
- net GND: now also C6.2, U10.2 (-Vin)
- net GND_OUT: now also U10.4 (-Vout)
Other:
- note added: "1. Q: [] 2. Q: [] 3. Q: [] 4. Q: [] 5. Q: []"
- note added: "105,50CZK"
- note added: "11,53CZK"
- note added: "42,35CZK"
- note added: "43,86CZK"
- note added: "GRAPHIC"
- note added: "Isolation: 1.5kV Output current: 400mA Output voltage: 5V Input voltage: 4.5V-5.5V Output power: 2W BUILT IN SHORT CIRCUIT PROTECTION"
- note added: "Max If: 50mA Reverse voltage: 6V Forward voltage: 1.2V-1.4V"
- note added: "Molex 9Pin header, 3.5mm Plug (female conn): 39503-3009"
- note added: "Output voltage: 3.3V Output current: 1A Max Input voltage: 12V Quiescent Current: 6mA"
- note added: "Termination resistor"
- note added: "Vf = 1.2V If = 20mA Vcc = 3.3V (RPi) R = (Vcc - Vf) / If R = 105R ~ 120R If [120R] = 17.5mA"
- note removed: "1. Q: Does the RS-485 have to be on its own separeted connector (twisted pair) 2. Q: 3. Q: 4. Q: 5. Q: []"
- note removed: "15,71CZK"
- note removed: "34,83CZK"
- note removed: "36,84CZK"
- note removed: "39,85CZK"
- note removed: "A zener diode can protect against overvoltage"
- note removed: "CIRCUIT PROTECTION"
- note removed: "I think we dont need it at all: Cost inneffective."
- note removed: "Isolation: 1.5kV Output current max: 200mA Voltage input: 4.5V-5.5V"
- note removed: "REVERSE POL. PROTECTION"
- note removed: "RS-485 max speed is 10Mb/s"
- note removed: "SCRAPPED"
- note removed: "TO-DO: - Change all of the logic to 3.3V logic - Can user error cause overvoltage on the gpio pin? (optocouplers) - Come up with a solution for 3.3V logic switch"
- note removed: "Vf = 1.2V If = 20mA Vcc = 3.3V (RPi) R = (Vcc - Vf) / If R = 105R ~ 120R If [120] = 17.5mA"
- note removed: "low Rds on"
- moved on the sheet: H1, H2, H3, H4, J1, J2
