File: IoTGW_Isolation/IoTGW_Isolation.kicad_pcb (KiCad board)
At the start: 2 copper layers, 40 x 48.5 mm, 35 parts, among them J1 39502-1009, J2 39502-1009, U10 TBA2-0511, U2 NCP1117-3.3, U3 LTV-817S, U4 LTV-817S, U5 LTV-817S, U6 LTV-817S, U7 LTV-817S, U8 LTV-817S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

Commit message: last update, plot of IoTGW isolation
Routing:
- net GND_OUT: track 5.97 -> 4.14 mm
- net Net-(R8-Pad1): track 27.8 -> 28.5 mm
- net +3.3V_OUT: track 40.2 -> 39.6 mm
